File: SoM/FPGA_TOP.kicad_sch (KiCad schematic)
At the start: 44 parts, among them U1 CCGM1A1, X1 ECS-5032MV

Commit message: Migrate project files to KiCad 10 format
Re-saved all schematics, the PCB and the SOP-8 footprint with
KiCad 10 (generator_version 9.0 -> 10.0). No components, nets,
placements or values were changed - this only updates the file
schema (new default fields, refreshed UUIDs) that KiCad 10 adds
on save.
Parts:
- JP9: value ~ -> (none)
- U1: footprint Package_BGA:BGA-324_15.0x15.0mm_Layout18x18_P0.8mm_Ball0.45mm_Pad0.4mm_NSMD -> ccsom_Footprint_lib:BGA-324_15x15mm_Layout18x18_P0.8mm
